Commit message: added URDF and Launch files

File: src/arduinobot_description/urdf/arduinobot.urdf.xacro (robot description, xacro)
@@ -1,12 +1,121 @@
 <?xml version="1.0"?>
 <robot name="arduinobot" xmlns:xacro="http://www.ros.org/wiki/xacro">
-<link name="world"/>
-<link name="base_link">
-    <visual>
+    <xacro:property name="effort" value="30.0"/>
+    <xacro:property name="velocity" value="30.0"/>
+    <link name="world"/>
+    <link name="base_link">
+        <visual>
+            <geometry>
+                <mesh filename="package://arduinobot_description/meshes/basement.STL" scale="0.01 0.01 0.01"/>
+            </geometry>
+            <origin xyz="-0.47 -0.45 0" rpy="0 0 0"/>
+        </visual>
+    </link>
+    <joint name="world_base_joint" type="fixed">
+        <parent link="world"/>
+        <child link="base_link"/>
         <origin xyz="0 0 0" rpy="0 0 0"/>
-        <geometry>
-            <mesh filename="package://arduinobot_description/meshes/basement.STL" scale="0.1 0.1 0.1"/>
-        </geometry>
-    </visual>
-</link>
+    </joint>
+    <link name="base_plate_link">
+        <visual>
+            <geometry>
+                <mesh filename="package://arduinobot_description/meshes/base_plate.STL" scale="0.01 0.01 0.01"/>
+            </geometry>
+            <origin xyz="-0.39 -0.39 -0.56" rpy="0 0 0"/>
+        </visual>
+    </link>
+    <joint name="base_base_plate_joint" type="revolute">
+        <parent link="base_link"/>
+        <child link="base_plate_link"/>
+        <origin xyz="0 0 0.307" rpy="0 0 0"/>
+        <axis xyz="0 0 1"/>
+        <limit lower="-${pi/2.0}" upper="${pi/2.0}" effort="${effort}" velocity="${velocity}"/>
+    </joint>
+    <link name="forward_drive_arm_link">
+        <visual>
+            <geometry>
+                <mesh filename="package://arduinobot_description/meshes/forward_drive_arm.STL" scale="0.01 0.01 0.01"/>
+            </geometry>
+            <origin xyz="0.19 0.06 -0.08" rpy="0 -${pi/2.0} ${pi/2.0}"/>
+        </visual>
+    </link>
+    <joint name="base_plate_forward_drive_arm_joint" type="revolute">
+        <parent link="base_plate_link"/>
+        <child link="forward_drive_arm_link"/>
+        <origin xyz="-0.02 0 0.35" rpy="0 0 0"/>
+        <axis xyz="1 0 0"/>
+        <limit lower="-${pi/2.0}" upper="${pi/2.0}" effort="${effort}" velocity="${velocity}"/>
+    </joint>
+     <link name="horizontal_arm_link">
+        <visual>
+            <geometry>
+                <mesh filename="package://arduinobot_description/meshes/horizontal_arm.STL" scale="0.01 0.01 0.01"/>
+            </geometry>
+            <origin xyz="-0.03 -0.4 -0.06" rpy="${pi/2.0} 0 ${pi/2.0}"/>
+        </visual>
+    </link>
+    <joint name="forward_horizontal_arm_joint" type="revolute">
+        <parent link="forward_drive_arm_link"/>
+        <child link="horizontal_arm_link"/>
+        <origin xyz="0 0 0.8" rpy="0 0 0"/>
+        <axis xyz="1 0 0"/>
+        <limit lower="-${pi/2.0}" upper="${pi/2.0}" effort="${effort}" velocity="${velocity}"/>
+    </joint>
+    <link name="claw_support_link">
+        <visual>
+            <geometry>
+                <mesh filename="package://arduinobot_description/meshes/claw_support.STL" scale="0.01 0.01 0.01"/>
+            </geometry>
+            <origin xyz="0 -0.05 -0.15" rpy="0 0 ${pi/2.0}"/>
+        </visual>
+    </link>
+    <joint name="horizontal_arm_claw_joint" type="fixed">
+        <parent link="horizontal_arm_link"/>
+        <child link="claw_support_link"/>
+        <origin xyz="0 0.82 0" rpy="0 0 0"/>
+    </joint>
+    <link name="gripper_right_link">
+        <visual>
+            <geometry>
+                <mesh filename="package://arduinobot_description/meshes/right_finger.STL" scale="0.01 0.01 0.01"/>
+            </geometry>
+            <origin xyz="-0.1 0.5 -0.1" rpy="0 0 -${pi/2.0}"/>
+        </visual>
+    </link>
+    <joint name="claw_gripper_right_joint" type="revolute">
+        <parent link="claw_support_link"/>
+        <child link="gripper_right_link"/>
+        <origin xyz="-0.04 0.13 -0.1" rpy="0 0 0"/>
+        <axis xyz="0 0 1"/>
+        <limit lower="-${pi/2.0}" upper="0.0" effort="${effort}" velocity="${velocity}"/>
+    </joint>
+     <link name="gripper_left_link">
+        <visual>
+            <geometry>
+                <mesh filename="package://arduinobot_description/meshes/left_finger.STL" scale="0.01 0.01 0.01"/>
+            </geometry>
+            <origin xyz="-0.04 0.5 -0.1" rpy="0 0 -${pi/2.0}"/>
+        </visual>
+    </link>
+    <joint name="claw_gripper_left_joint" type="revolute">
+        <parent link="claw_support_link"/>
+        <child link="gripper_left_link"/>
+        <origin xyz="-0.22 0.13 -0.1" rpy="0 0 0"/>
+        <axis xyz="0 0 1"/>
+        <limit lower="0.0" upper="${pi/2.0}" effort="${effort}" velocity="${velocity}"/>
+        <mimic joint="claw_gripper_right_joint" multiplier="-1"/>
+    </joint>
+    <link name="rgb_camera_link">
+        <visual>
+            <geometry>
+                <mesh filename="package://arduinobot_description/meshes/pi_camera.STL" scale="0.01 0.01 0.01"/>
+            </geometry>
+            <origin xyz="-0.1 0.125 0.15" rpy="-${pi/2.0} 0 -${pi/2.0}"/>
+        </visual>
+    </link>
+    <joint name="base_rgb_camera_joint" type="fixed">
+        <parent link="base_link"/>
+        <child link="rgb_camera_link"/>
+        <origin xyz="0 0.5 0.2" rpy="0 -0.5 ${pi/2.0}"/>
+    </joint>
 </robot>
